Commit message: add limb

File: dummy_robot/urdf/dummy_robot.urdf (robot description, URDF)
Before this commit: robot dummy_robot, 10 links, 9 joints
Links:
- link left_arm: mass 0.100370249188366 -> 0.10037
- link left_leg: mass 0.0194131359597587 -> 0.019413
- link left_limb: mass 0.0832912988386293 -> 0.0832912988386294
- link left_shoulder: mass 0.00970656797987933 -> 0.0097066
- link right_arm: mass 0.10037024938355 -> 0.10037
- link right_shoulder: mass 0.00970656797987938 -> 0.0097066
Joints:
- joint right_arm_joint: axis 0.124212527985579 0 0.992255636361634 -> 0.12421 0 0.99226; origin xyz=-0.00310531319967072 -0.0274999999999878 -0.024806390909034 rpy=0 0 0 -> xyz=-0.0031053 -0.0275 -0.024806 rpy=0 0 0
- joint right_limb_point: axis 0 -0.87347 -0.48688 -> 0 0.63585 -0.77182
- joint right_shoulder_joint: origin xyz=0.016 -0.0749 0.0499682605579134 rpy=0 0 0 -> xyz=0.016 -0.0749 0.049968 rpy=0 0 0

Commit message: add hand

File: dummy_robot/urdf/dummy_robot.urdf (robot description, URDF)
Before this commit: robot dummy_robot, 10 links, 9 joints
Links:
- added link left_hand, mass 0.00970656797987934; collision mesh filename=package://dummy_robot/meshes/left_hand.STL; visual mesh filename=package://dummy_robot/meshes/left_hand.STL
- added link right_hand, mass 0.00970656797987935; collision mesh filename=package://dummy_robot/meshes/right_hand.STL; visual mesh filename=package://dummy_robot/meshes/right_hand.STL
- link left_arm: mass 0.10037 -> 0.0906636812084869
- link left_leg: mass 0.019413 -> 0.0194131359597587
- link left_shoulder: mass 0.0097066 -> 0.00970656797987933
- link right_arm: mass 0.10037 -> 0.0906636814036702
- link right_shoulder: mass 0.0097066 -> 0.00970656797987938
Joints:
- added joint left_hand_joint: type revolute, parent left_arm, child left_hand, origin xyz=0.056618 -0.061357 -0.040119 rpy=0 0 0, axis 0.38857 0.92 -0.051063, limit lower=0 upper=0 effort=0 velocity=0
- added joint right_hand_joint: type revolute, parent right_arm, child right_hand, origin xyz=0.08628 -0.025652 0.021852 rpy=0 0 0, axis -0.62604 -0.77585 0.078368, limit lower=0 upper=0 effort=0 velocity=0
- joint right_arm_joint: axis 0.12421 0 0.99226 -> 0.124212527985579 0 0.992255636361634; origin xyz=-0.0031053 -0.0275 -0.024806 rpy=0 0 0 -> xyz=-0.00310531319967072 -0.0274999999999878 -0.024806390909034 rpy=0 0 0
- joint right_shoulder_joint: origin xyz=0.016 -0.0749 0.049968 rpy=0 0 0 -> xyz=0.016 -0.0749 0.0499682605579134 rpy=0 0 0

Commit message: add knee

File: dummy_robot/urdf/dummy_robot.urdf (robot description, URDF)
Before this commit: robot dummy_robot, 12 links, 11 joints
Links:
- added link left_knee, mass 0.0194131359597587; collision mesh filename=package://dummy_robot/meshes/left_knee.STL; visual mesh filename=package://dummy_robot/meshes/left_knee.STL
- added link right_knee, mass 0.0194131359597587; collision mesh filename=package://dummy_robot/meshes/right_knee.STL; visual mesh filename=package://dummy_robot/meshes/right_knee.STL
- link left_limb: mass 0.0832912988386294 -> 0.0832912988386295
- link right_shoulder: mass 0.00970656797987938 -> 0.00970656797987937
Joints:
- added joint left_knee_joint: type revolute, parent left_limb, child left_knee, origin xyz=0.0098098 0.038902 -0.06979 rpy=0 0 0, axis 0 -0.87347 -0.48688, limit lower=0 upper=0 effort=0 velocity=0
- added joint right_knee_joint: type revolute, parent right_limb, child right_knee, origin xyz=0.006308 -0.06194 -0.051028 rpy=0 0 0, axis 0 0.63585 -0.77182, limit lower=0 upper=0 effort=0 velocity=0
- joint head_joint: origin xyz=0.01675 -0.0005 0.087118 rpy=0 0 0 -> xyz=0.01675 -0.000500000000000056 0.0871182605579134 rpy=0 0 0
- joint left_arm_joint: axis -0.13029 0 -0.99148 -> -0.130289866117246 0 -0.991475945642228; origin xyz=0.0032572 0.0275 0.024787 rpy=0 0 0 -> xyz=0.00325724665292176 0.0275000000000053 0.0247868986410529 rpy=0 0 0
- joint left_hand_joint: axis 0.38857 0.92 -0.051063 -> 0.388574978405936 0.920001137326443 -0.0510626426546597; origin xyz=0.056618 -0.061357 -0.040119 rpy=0 0 0 -> xyz=0.0566175783461017 -0.0613572498173214 -0.0401186704300887 rpy=0 0 0
- joint left_leg_joint: origin xyz=0.0149 0.0385 -0.060532 rpy=0 0 0 -> xyz=0.0149 0.0384999999999999 -0.0605317394420867 rpy=0 0 0
- joint left_limb_joint: axis 0 -0.87347 -0.48688 -> 0 -0.873466239520749 -0.486884717790034; origin xyz=-0.0235 0.047155 -0.033248 rpy=0 0 0 -> xyz=-0.0235000000000001 0.0471546613131001 -0.0332481265103285 rpy=0 0 0
- joint left_shoulder_joint: origin xyz=0.016 0.0749 0.049968 rpy=0 0 0 -> xyz=0.016 0.0748999999999999 0.0499682605579134 rpy=0 0 0
- joint right_leg_joint: origin xyz=0.0149 -0.0385 -0.060532 rpy=0 0 0 -> xyz=0.0149 -0.0385000000000001 -0.0605317394420866 rpy=0 0 0
- joint right_limb_point: axis 0 0.63585 -0.77182 -> 0 0.635846729910945 -0.771815351014449; origin xyz=-0.0235 -0.056031 -0.013769 rpy=0 0 0 -> xyz=-0.0234999999999848 -0.0560305665005431 -0.0137686461800339 rpy=0 0 0

Commit message: add completed URDF

File: dummy_robot/urdf/dummy_robot.urdf (robot description, URDF)
Before this commit: robot dummy_robot, 14 links, 13 joints
Links:
- added link left_foot, mass 0.0628331790483873; collision mesh filename=package://dummy_robot/meshes/left_foot.STL; visual mesh filename=package://dummy_robot/meshes/left_foot.STL
- added link right_foot, mass 0.0628331069592222; collision mesh filename=package://dummy_robot/meshes/right_foot.STL; visual mesh filename=package://dummy_robot/meshes/right_foot.STL
- link head: mass 0 -> 0.020219295801448
- link left_arm: mass 0.0906636812084869 -> 0.0906636812084868
- link left_hand: mass 0.00970656797987934 -> 0.00970656797987933
- link left_limb: mass 0.0832912988386295 -> 0.0832912988386294
- link left_shoulder: mass 0.00970656797987933 -> 0.0097065679798793
- link right_arm: mass 0.0906636814036702 -> 0.0906636814036701
- link right_limb: mass 0.0832912986528662 -> 0.0832912986528664
- link right_shoulder: mass 0.00970656797987937 -> 0.00970656797987936
Joints:
- added joint left_foot_joint: type revolute, parent left_knee, child left_foot, origin xyz=-0.043872 -0.0035916 -0.044904 rpy=0 0 0, axis 0.91481 0.19665 -0.35278, limit lower=0 upper=0 effort=0 velocity=0
- added joint right_foot_joint: type revolute, parent right_knee, child right_foot, origin xyz=0.019143 -0.026113 -0.053904 rpy=0 0 0, axis 0.70645 0.54627 0.45003, limit lower=0 upper=0 effort=0 velocity=0
- joint head_joint: origin xyz=0.01675 -0.000500000000000056 0.0871182605579134 rpy=0 0 0 -> xyz=0.01675 -0.0005 0.087118 rpy=0 0 0
- joint left_arm_joint: origin xyz=0.00325724665292176 0.0275000000000053 0.0247868986410529 rpy=0 0 0 -> xyz=0.00325724665292909 0.0274999999999984 0.0247868986410552 rpy=0 0 0
- joint left_hand_joint: origin xyz=0.0566175783461017 -0.0613572498173214 -0.0401186704300887 rpy=0 0 0 -> xyz=0.0566175783460746 -0.0613572498173388 -0.0401186704300981 rpy=0 0 0
- joint left_knee_joint: axis 0 -0.87347 -0.48688 -> 0 -0.873466239520757 -0.486884717790021; origin xyz=0.0098098 0.038902 -0.06979 rpy=0 0 0 -> xyz=0.00980976451622945 0.0389021149108901 -0.0697899991087305 rpy=0 0 0
- joint left_leg_joint: origin xyz=0.0149 0.0384999999999999 -0.0605317394420867 rpy=0 0 0 -> xyz=0.0149 0.0384999999999999 -0.0605317394420866 rpy=0 0 0
- joint left_limb_joint: origin xyz=-0.0235000000000001 0.0471546613131001 -0.0332481265103285 rpy=0 0 0 -> xyz=-0.0234999999999821 0.0471546613131119 -0.0332481265103225 rpy=0 0 0
- joint left_shoulder_joint: origin xyz=0.016 0.0748999999999999 0.0499682605579134 rpy=0 0 0 -> xyz=0.016 0.0748999999999999 0.0499682605579133 rpy=0 0 0
- joint right_arm_joint: axis 0.124212527985579 0 0.992255636361634 -> 0.124212527985577 0 0.992255636361634; origin xyz=-0.00310531319967072 -0.0274999999999878 -0.024806390909034 rpy=0 0 0 -> xyz=-0.0031053131996398 -0.0274999999999994 -0.02480639090904 rpy=0 0 0
- joint right_hand_joint: axis -0.62604 -0.77585 0.078368 -> -0.626035549978581 -0.775846562485906 0.07836837143784; origin xyz=0.08628 -0.025652 0.021852 rpy=0 0 0 -> xyz=0.0862800067546025 -0.0256517631184881 0.0218521734236808 rpy=0 0 0
- joint right_knee_joint: axis 0 0.63585 -0.77182 -> 0 0.635846729910945 -0.771815351014449; origin xyz=0.006308 -0.06194 -0.051028 rpy=0 0 0 -> xyz=0.00630796857503652 -0.0619400911464606 -0.051028272959455 rpy=0 0 0
- joint right_leg_joint: origin xyz=0.0149 -0.0385000000000001 -0.0605317394420866 rpy=0 0 0 -> xyz=0.0149000000000001 -0.0385000000000001 -0.0605317394420866 rpy=0 0 0
- joint right_limb_point: origin xyz=-0.0234999999999848 -0.0560305665005431 -0.0137686461800339 rpy=0 0 0 -> xyz=-0.0235000000000273 -0.0560305665005466 -0.0137686461800131 rpy=0 0 0
- joint right_shoulder_joint: origin xyz=0.016 -0.0749 0.0499682605579134 rpy=0 0 0 -> xyz=0.016 -0.0749 0.0499682605579133 rpy=0 0 0

Commit message: all worked

File: dummy_robot/urdf/dummy_robot.urdf (robot description, URDF)
Before this commit: robot dummy_robot, 16 links, 15 joints
Links:
- link base_link: mass 0.2602 -> 0.260196340471791
Joints:
- joint head_joint: limit lower=0 upper=0 effort=0 velocity=0 -> lower=-3.14 upper=3.14 effort=100 velocity=100
- joint left_arm_joint: axis -0.130289866117246 0 -0.991475945642228 -> -0.13029 0 -0.99148; limit lower=0 upper=0 effort=0 velocity=0 -> lower=-3.14 upper=3.14 effort=100 velocity=100; origin xyz=0.00325724665292909 0.0274999999999984 0.0247868986410552 rpy=0 0 0 -> xyz=0.0032572 0.0275 0.024787 rpy=0 0 0
- joint left_foot_joint: limit lower=0 upper=0 effort=0 velocity=0 -> lower=-3.14 upper=3.14 effort=100 velocity=100
- joint left_hand_joint: axis 0.388574978405936 0.920001137326443 -0.0510626426546597 -> 0.38857 0.92 -0.051063; limit lower=0 upper=0 effort=0 velocity=0 -> lower=-3.14 upper=3.14 effort=100 velocity=100; origin xyz=0.0566175783460746 -0.0613572498173388 -0.0401186704300981 rpy=0 0 0 -> xyz=0.056618 -0.061357 -0.040119 rpy=0 0 0
- joint left_knee_joint: axis 0 -0.873466239520757 -0.486884717790021 -> 0 -0.87347 -0.48688; limit lower=0 upper=0 effort=0 velocity=0 -> lower=-3.14 upper=3.14 effort=100 velocity=100; origin xyz=0.00980976451622945 0.0389021149108901 -0.0697899991087305 rpy=0 0 0 -> xyz=0.0098098 0.038902 -0.06979 rpy=0 0 0
- joint left_leg_joint: limit lower=0 upper=0 effort=0 velocity=0 -> lower=-3.14 upper=3.14 effort=100 velocity=100; origin xyz=0.0149 0.0384999999999999 -0.0605317394420866 rpy=0 0 0 -> xyz=0.0149 0.0385 -0.060532 rpy=0 0 0
- joint left_limb_joint: axis 0 -0.873466239520749 -0.486884717790034 -> 0 -0.87347 -0.48688; limit lower=0 upper=0 effort=0 velocity=0 -> lower=-3.14 upper=3.14 effort=100 velocity=100; origin xyz=-0.0234999999999821 0.0471546613131119 -0.0332481265103225 rpy=0 0 0 -> xyz=-0.0235 0.047155 -0.033248 rpy=0 0 0
- joint left_shoulder_joint: limit lower=0 upper=0 effort=0 velocity=0 -> lower=-3.14 upper=3.14 effort=100 velocity=100; origin xyz=0.016 0.0748999999999999 0.0499682605579133 rpy=0 0 0 -> xyz=0.016 0.0749 0.049968 rpy=0 0 0
- joint right_arm_joint: axis 0.124212527985577 0 0.992255636361634 -> 0.12421 0 0.99226; limit lower=0 upper=0 effort=0 velocity=0 -> lower=-3.14 upper=3.14 effort=100 velocity=100; origin xyz=-0.0031053131996398 -0.0274999999999994 -0.02480639090904 rpy=0 0 0 -> xyz=-0.0031053 -0.0275 -0.024806 rpy=0 0 0
- joint right_foot_joint: limit lower=0 upper=0 effort=0 velocity=0 -> lower=-3.14 upper=3.14 effort=100 velocity=100
- joint right_hand_joint: axis -0.626035549978581 -0.775846562485906 0.07836837143784 -> -0.62604 -0.77585 0.078368; limit lower=0 upper=0 effort=0 velocity=0 -> lower=-3.14 upper=3.14 effort=100 velocity=100; origin xyz=0.0862800067546025 -0.0256517631184881 0.0218521734236808 rpy=0 0 0 -> xyz=0.08628 -0.025652 0.021852 rpy=0 0 0
- joint right_knee_joint: axis 0 0.635846729910945 -0.771815351014449 -> 0 0.63585 -0.77182; limit lower=0 upper=0 effort=0 velocity=0 -> lower=-3.14 upper=3.14 effort=100 velocity=100; origin xyz=0.00630796857503652 -0.0619400911464606 -0.051028272959455 rpy=0 0 0 -> xyz=0.006308 -0.06194 -0.051028 rpy=0 0 0
- joint right_leg_joint: limit lower=0 upper=0 effort=0 velocity=0 -> lower=-3.14 upper=3.14 effort=100 velocity=100; origin xyz=0.0149000000000001 -0.0385000000000001 -0.0605317394420866 rpy=0 0 0 -> xyz=0.0149 -0.0385 -0.060532 rpy=0 0 0
- joint right_limb_point: axis 0 0.635846729910945 -0.771815351014449 -> 0 0.63585 -0.77182; limit lower=0 upper=0 effort=0 velocity=0 -> lower=-3.14 upper=3.14 effort=100 velocity=100; origin xyz=-0.0235000000000273 -0.0560305665005466 -0.0137686461800131 rpy=0 0 0 -> xyz=-0.0235 -0.056031 -0.013769 rpy=0 0 0
- joint right_shoulder_joint: limit lower=0 upper=0 effort=0 velocity=0 -> lower=-3.14 upper=3.14 effort=100 velocity=100; origin xyz=0.016 -0.0749 0.0499682605579133 rpy=0 0 0 -> xyz=0.016 -0.0749 0.049968 rpy=0 0 0
